File: pcb/BlinkyBoard.brd (EAGLE design)
At the start: 25.2 x 10 mm, 27 parts, among them Q1 16 MHz

Commit message: Fix label: Analog input is actually on A9, not 11!
Connections:
- net A10 renamed A9
Other:
- board text added: "A9"
- board text removed: "A11"
Changed lines of the file:
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@@
 <text x="20.75" y="2" size="0.75" layer="26" font="vector" ratio="15" rot="MR0" align="center">GND</text>
 <text x="20.5" y="8.75" size="0.75" layer="26" font="vector" ratio="15" rot="MR0" align="bottom-center">5V</text>
-<text x="20.75" y="5" size="0.75" layer="26" font="vector" ratio="15" rot="MR0" align="center">A11</text>
+<text x="20.75" y="5" size="0.75" layer="26" font="vector" ratio="15" rot="MR0" align="center">A9</text>
 <text x="4.35" y="6.25" size="0.75" layer="26" font="vector" ratio="15" rot="MR0" align="center">D7</text>
 <text x="4.65" y="3.75" size="0.75" layer="26" font="vector" ratio="15" rot="MR0" align="center">D11</text>
@@
 <wire x1="9.14" y1="7.75" x2="10.225" y2="7.75" width="0.254" layer="1"/>
 </signal>
-<signal name="A10">
+<signal name="A9">
 <contactref element="U$2" pad="29"/>
 <via x="18.8" y="6.1" extent="1-16" drill="0.35"/>
